File: B.E.M-sbc3x/B.E.M-sbc3x.sch (KiCad schematic (older format))
At the start: 7 parts, among them J1 Screw_Terminal_01x02, U1 6822, U2 6822, U3 MC68A09, U4 TC55257PL-12, U5 27256, U6 DM74S571

Commit message: Almost finnished with the schema and layout. Only some jumpers are not yet mapped out. For the PCB layout is only component placement is done, no routing
Parts:
- added B1: Battery_Cell, B.E.M:Battery_3.6v, symbol Device:Battery_Cell
- added C11: 10uF, symbol Device:CP_Small
- added C14: 100n, Capacitor_THT:C_Rect_L7.0mm_W2.0mm_P5.00mm, symbol Device:C
- added C15: 10n, Capacitor_THT:C_Rect_L7.0mm_W2.0mm_P5.00mm, symbol Device:C
- added C16: 100pF, Capacitor_THT:C_Rect_L7.0mm_W2.0mm_P5.00mm, symbol Device:C
- added C17, C18: 22p, Capacitor_THT:C_Rect_L7.0mm_W2.0mm_P5.00mm, symbol Device:C
- added C2: 22P, Capacitor_THT:C_Rect_L7.0mm_W2.0mm_P5.00mm, symbol Device:C
- added CN1, CN2, CN3: Conn_02x13_Odd_Even, Connector_PinSocket_2.54mm:PinSocket_2x13_P2.54mm_Vertical, symbol Connector_Generic:Conn_02x13_Odd_Even
- added CN5, CN6: Conn_02x05_Odd_Even, Connector_PinSocket_2.54mm:PinSocket_2x05_P2.54mm_Vertical, symbol Connector_Generic:Conn_02x05_Odd_Even
- added CT1: 30pF, Capacitor_THT:C_Rect_L7.2mm_W5.5mm_P5.00mm_FKS2_FKP2_MKS2_MKP2, symbol Device:C_Variable
- added D1: 1N4148, Diode_THT:D_A-405_P7.62mm_Horizontal, symbol Device:D
- added D2: 1N4148, Diode_THT:D_5W_P10.16mm_Horizontal, symbol Device:D
- added EXP1: Exp, Connector_PinHeader_2.54mm:PinHeader_1x08_P2.54mm_Vertical, symbol Connector_Generic:Conn_01x08
- added JP1, JP12, JP13, JP14, JP15, JP16, JP17, JP18, JP19, JP2, JP20, JP21, JP3: Jumper_NO_Small, Resistor_THT:R_Axial_DIN0204_L3.6mm_D1.6mm_P1.90mm_Vertical, symbol Device:Jumper_NO_Small
- added JP10, JP11, JP22, JP6, JP7, JP8, JP9: Jumper_3_Open, symbol Jumper:Jumper_3_Open
- added JP23, JP4, JP5: Jumper_3_Open, Connector_PinHeader_2.54mm:PinHeader_1x03_P2.54mm_Vertical, symbol Jumper:Jumper_3_Open
- added Q1: BD136, Package_TO_SOT_THT:TO-126-3_Vertical, symbol Transistor_BJT:BD136
- added Q2: BC556, Package_TO_SOT_THT:TO-92_Inline, symbol Transistor_BJT:BC556
- added Q3, Q4, Q5, Q6, Q7, Q8: BC547, Package_TO_SOT_THT:TO-92_Inline, symbol Transistor_BJT:BC547
- added R1, R13, R3, R4: 10K, Resistor_THT:R_Axial_DIN0207_L6.3mm_D2.5mm_P10.16mm_Horizontal, symbol Device:R
- added R10, R14, R15, R8, R9: 3.3K, Resistor_THT:R_Axial_DIN0207_L6.3mm_D2.5mm_P10.16mm_Horizontal, symbol Device:R
- added R11: 220K, Resistor_THT:R_Axial_DIN0207_L6.3mm_D2.5mm_P10.16mm_Horizontal, symbol Device:R
- added R12: 22K, Resistor_THT:R_Axial_DIN0207_L6.3mm_D2.5mm_P10.16mm_Horizontal, symbol Device:R
- added R2, R6, R7: 1K, Resistor_THT:R_Axial_DIN0207_L6.3mm_D2.5mm_P10.16mm_Horizontal, symbol Device:R
- added R5: 100, Resistor_THT:R_Axial_DIN0207_L6.3mm_D2.5mm_P10.16mm_Horizontal, symbol Device:R
- added RN1, RN5: 10K, Resistor_THT:R_Array_SIP10, symbol Device:R_Network09
- added RN2: 2k, Resistor_THT:R_Array_SIP8, symbol Device:R_Network07
- added RN3: 3.3K, Resistor_THT:R_Array_SIP4, symbol Device:R_Network03
- added RN4: 10K, Resistor_THT:R_Array_SIP8, symbol Device:R_Network07
- added RN6: 3.3K, Resistor_THT:R_Array_SIP6, symbol Device:R_Network05
- added U1: TC55257PL-12, Package_DIP:DIP-28_W15.24mm, symbol B.E.M-sbc3x:TC55257PL-12
- added U10: 74LS00, Package_DIP:DIP-14_W7.62mm_Socket, symbol 74xx:74LS00
- added U11: 74HC04, symbol 74xx:74HC04
- added U12: CD4060BCN, Package_DIP:DIP-16_W7.62mm_LongPads, symbol B.E.M-sbc3x:CD4060BCN
- added U13: 6822, Package_DIP:DIP-40_W15.24mm, symbol Interface:6822
- added U15: MM58274BN, Package_DIP:DIP-16_W7.62mm_Socket, symbol B.E.M-sbc3x:MM58274BN
- added U6: TL7705ACPSR, Package_DIP:DIP-8_W7.62mm_Socket, symbol Power_Supervisor:TL7705ACPSR
- added U7: INS2651, Package_DIP:DIP-28_W15.24mm_Socket, symbol B.E.M-sbc3x:INS2651
- added U9: 74LS42, Package_DIP:DIP-16_W7.62mm_Socket, symbol 74xx:74LS42
- added X1: 32.768, Crystal:Crystal_DS26_D2.0mm_L6.0mm_Vertical, symbol Device:Crystal
- added X2: 5.0688, Crystal:Crystal_HC18-U_Horizontal, symbol Device:Crystal
- added X3: 4.000, Crystal:Crystal_HC18-U_Horizontal, symbol Device:Crystal
- added ZD1: D_Zener, symbol Device:D_Zener
- renumbered U2 to U14, U4 to U2, U5 to U3, U3 to U4, U1 to U5, U6 to U8
Connections:
- net labels added: BrC, C1-1, C1-10, C1-11, C1-12, C1-13, C1-14, C1-15, C1-16, C1-17, C1-18, C1-19, C1-2, C1-20, C1-21, C1-22, C1-23, C1-24, C1-25, C1-26, C1-3, C1-4, C1-5, C1-6, C1-7, C1-8, C1-9, C2-1, C2-10, C2-11, C2-12, C2-13, C2-14, C2-15, C2-16, C2-17, C2-18, C2-19, C2-2, C2-20, C2-21, C2-22, C2-23, C2-24, C2-25, C2-26, C2-3, C2-4, C2-5, C2-6, C2-7, C2-8, C2-9, C3-1, C3-10, C3-11, C3-12, C3-13, C3-14, C3-15, C3-16, C3-17, C3-18, C3-19, C3-2, C3-20, C3-21, C3-22, C3-23, C3-24, C3-25, C3-26, C3-3, C3-4, C3-5, C3-6, C3-7, C3-8, C3-9, C5-1, C5-10, C5-2, C5-3, C5-4, C5-5, C5-6, C5-7, C5-8, C5-9, C6-1, C6-10, C6-2, C6-3, C6-4, C6-5, C6-6, C6-7, C6-8, C6-9, E, RW, VCC, VDD
- wire segments 103 -> 693
Other:
- note added: "B.E.M Single Board Computer 3X"
- note added: "F"
- note added: "I"
- note added: "NP"
- note added: "Timer\nBatBacked"
- moved on the sheet: J1, U14, U2, U3, U4, U5, U8

Commit message: All connectors are mapped, daughter DATAC-1A mapped, components all placed on PCB, HD46508PA added to library
Parts:
- removed C14: 100n, Capacitor_THT:C_Rect_L7.0mm_W2.0mm_P5.00mm, symbol Device:C
- removed C15: 10n, Capacitor_THT:C_Rect_L7.0mm_W2.0mm_P5.00mm, symbol Device:C
- removed C16: 100pF, Capacitor_THT:C_Rect_L7.0mm_W2.0mm_P5.00mm, symbol Device:C
- removed C17, C18: 22p, Capacitor_THT:C_Rect_L7.0mm_W2.0mm_P5.00mm, symbol Device:C
- removed C2: 22P, Capacitor_THT:C_Rect_L7.0mm_W2.0mm_P5.00mm, symbol Device:C
- removed CT1: 30pF, Capacitor_THT:C_Rect_L7.2mm_W5.5mm_P5.00mm_FKS2_FKP2_MKS2_MKP2, symbol Device:C_Variable
- added C1, C10, C12, C13, C14, C15, C3, C4, C5, C6, C7, C8: 100nF, Capacitor_THT:C_Rect_L7.0mm_W2.0mm_P5.00mm, symbol Device:C_Small
- added C16: 100pF, Capacitor_THT:C_Disc_D3.4mm_W2.1mm_P2.50mm, symbol Device:C_Small
- added C17, C18, C2: 22pF, Capacitor_THT:C_Disc_D3.4mm_W2.1mm_P2.50mm, symbol Device:C_Small
- added C9: 10uF, symbol Device:CP_Small
- added CT1: 6-30pF, Capacitor_THT:C_Disc_D6.0mm_W4.4mm_P5.00mm, symbol Device:CTRIM_Small
- C11: footprint (none) -> Capacitor_THT:CP_Radial_Tantal_D4.5mm_P2.50mm
- JP10, JP11, JP6, JP7, JP8, JP9: footprint (none) -> Connector_PinHeader_2.54mm:PinHeader_1x03_P2.54mm_Vertical
Connections:
- wire segments 693 -> 866
Other:
- note added: "Plugin board"
- moved on the sheet: JP10, JP11, JP19, JP20, JP4, JP6, JP7, JP8, JP9, R15, R8, U10A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
